Commit message: added ur5 arm and 2 finger gripper

File: assets/desk/desk.urdf (robot description, URDF)
Before this commit: robot playroom_ec_desk, 12 links, 11 joints
Links:
- removed link Button1top
- removed link Button2top
- removed link Button3top
Joints:
- removed joint button1top_joint
- removed joint button2top_joint
- removed joint button3top_joint

Commit message: env test in progress
have strange oscillation on gripper when get close to deks... need to check. ALso slide does not seem to work / move - mayeb issues related

File: assets/desk/desk.urdf (robot description, URDF)
Before this commit: robot playroom_ec_desk, 9 links, 8 joints
Links:
- link Button1: mass 0.1 -> 0.01
- link Button2: mass 0.1 -> 0.01
- link Button3: mass 0.1 -> 0.01
- link Desk: mass 155 -> 554.5

File: assets/ur5/ur5.urdf (robot description, URDF)
Before this commit: robot ur5, 16 links, 15 joints
Joints:
- joint base_to_left_fingertip: limit lower=0 upper=0.03 effort=1.0 velocity=0.1 -> lower=0 upper=0.03 effort=1.0 velocity=3.2
- joint base_to_right_fingertip: limit lower=-0.03 upper=0.0 effort=1.0 velocity=0.1 -> lower=-0.03 upper=0.0 effort=1.0 velocity=3.2

Commit message: autoplay test_env complete task 0, 1, 2

File: assets/desk/desk.urdf (robot description, URDF)
Before this commit: robot playroom_ec_desk, 9 links, 8 joints
Links:
- link Desk: geometry visual mesh filename=meshes/StudyTable.stl scale=0.01 0.01 0.01
